File: hardware/IX01/IX01.brd (EAGLE design)
At the start: 23.5 x 23.5 mm, 15 parts, among them IC1 P82B715, IC2 P82B715

Commit message: IX01 for Seeedstudio
Parts:
- removed Z2: (no value), dp_devices:SOD-323F
- added C1: 100 nF, rcl:C0805
- moved R2 1.27 mm to (8.57, 7.94)
- moved R4 1.27 mm to (12.4, 7.94)
Connections:
- net GND: now also C1.2; no longer Z2.A
- net VCC: now also C1.1; no longer Z2.C
Routing:
- net VCC: track 101.1 -> 99.1 mm
- net SC1: track 28.0 -> 29.1 mm
- net GND: vias 2 -> 3
Changed lines of the file:
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@@
 <layer number="20" name="Dimension" color="15" fill="1" visible="yes" active="yes"/>
 <layer number="21" name="tPlace" color="14" fill="1" visible="yes" active="yes"/>
-<layer number="22" name="bPlace" color="13" fill="1" visible="yes" active="yes"/>
+<layer number="22" name="bPlace" color="13" fill="1" visible="no" active="yes"/>
 <layer number="23" name="tOrigins" color="15" fill="1" visible="yes" active="yes"/>
 <layer number="24" name="bOrigins" color="15" fill="1" visible="yes" active="yes"/>
 <layer number="25" name="tNames" color="7" fill="1" visible="yes" active="yes"/>
-<layer number="26" name="bNames" color="7" fill="1" visible="yes" active="yes"/>
+<layer number="26" name="bNames" color="7" fill="1" visible="no" active="yes"/>
 <layer number="27" name="tValues" color="7" fill="1" visible="yes" active="yes"/>
-<layer number="28" name="bValues" color="7" fill="1" visible="yes" active="yes"/>
+<layer number="28" name="bValues" color="7" fill="1" visible="no" active="yes"/>
 <layer number="29" name="tStop" color="7" fill="3" visible="yes" active="yes"/>
 <layer number="30" name="bStop" color="7" fill="6" visible="yes" active="yes"/>
@@
 <attribute name="VALUE" x="12.3825" y="20.0025" size="1.27" layer="27" rot="R90"/>
 </element>
-<element name="R2" library="rcl" package="R0805" value="" x="9.8425" y="7.9375" smashed="yes" rot="R270">
-<attribute name="NAME" x="12.22375" y="6.985" size="1.27" layer="25" font="vector" ratio="15" rot="R90"/>
-<attribute name="VALUE" x="7.3025" y="8.5725" size="1.27" layer="27" rot="R270"/>
+<element name="R2" library="rcl" package="R0805" value="" x="8.5725" y="7.9375" smashed="yes" rot="R270">
+<attribute name="NAME" x="9.68375" y="9.2075" size="1.27" layer="25" font="vector" ratio="15" rot="R270"/>
+<attribute name="VALUE" x="6.0325" y="8.5725" size="1.27" layer="27" rot="R270"/>
 </element>
 <element name="R3" library="rcl" package="R0805" value="" x="13.6525" y="20.6375" smashed="yes" rot="R90">
@@
 <attribute name="VALUE" x="16.1925" y="20.0025" size="1.27" layer="27" rot="R90"/>
 </element>
-<element name="R4" library="rcl" package="R0805" value="" x="13.6525" y="7.9375" smashed="yes" rot="R270">
-<attribute name="NAME" x="16.03375" y="6.985" size="1.27" layer="25" font="vector" ratio="15" rot="R90"/>
-<attribute name="VALUE" x="11.1125" y="8.5725" size="1.27" layer="27" rot="R270"/>
+<element name="R4" library="rcl" package="R0805" value="" x="12.3825" y="7.9375" smashed="yes" rot="R270">
+<attribute name="NAME" x="13.49375" y="9.2075" size="1.27" layer="25" font="vector" ratio="15" rot="R270"/>
+<attribute name="VALUE" x="9.8425" y="8.5725" size="1.27" layer="27" rot="R270"/>
 </element>
 <element name="IC2" library="dp_devices" package="SO-8" value="P82B715" x="11.43" y="14.2875" smashed="yes" rot="MR180">
@@
 <attribute name="VALUE" x="9.285" y="5.2275" size="1.27" layer="28" font="vector" ratio="10" rot="MR270"/>
 </element>
-<element name="Z2" library="dp_devices" package="SOD-323F" value="" x="16.51" y="4.1275" smashed="yes" rot="MR270">
-<attribute name="NAME" x="15.1925" y="2.37" size="1.27" layer="26" font="vector" ratio="15" rot="MR180"/>
-<attribute name="VALUE" x="18.81" y="5.2275" size="1.27" layer="28" font="vector" ratio="10" rot="MR270"/>
+<element name="C1" library="rcl" package="C0805" value="100 nF" x="16.1925" y="7.9375" smashed="yes" rot="R90">
+<attribute name="NAME" x="17.30375" y="9.2075" size="1.27" layer="25" font="vector" ratio="15" rot="R270"/>
 </element>
 </elements>
@@
 <contactref element="D4" pad="1"/>
 <contactref element="Z1" pad="A"/>
-<contactref element="Z2" pad="A"/>
+<contactref element="C1" pad="2"/>
+<wire x1="16.1925" y1="8.8875" x2="16.1925" y2="8.89" width="0.4064" layer="1"/>
+<via x="18.0975" y="10.4775" extent="1-16" drill="0.6" shape="square"/>
 </signal>
 <signal name="VCC">
@@
 <wire x1="1.27" y1="16.51" x2="1.27" y2="12.3825" width="0.4064" layer="16"/>
 <wire x1="1.27" y1="12.3825" x2="3.175" y2="10.4775" width="0.4064" layer="16"/>
-<wire x1="9.8425" y1="6.9875" x2="6.665" y2="6.9875" width="0.4064" layer="1"/>
+<wire x1="8.5725" y1="6.9875" x2="6.665" y2="6.9875" width="0.4064" layer="1"/>
 <wire x1="6.665" y1="6.9875" x2="3.175" y2="10.4775" width="0.4064" layer="1"/>
-<wire x1="13.6525" y1="6.9875" x2="9.8425" y2="6.9875" width="0.4064" layer="1"/>
-<wire x1="15.3875" y1="6.9875" x2="15.875" y2="6.9875" width="0.4064" layer="16"/>
-<wire x1="15.875" y1="6.9875" x2="16.83" y2="6.9875" width="0.4064" layer="16"/>
+<wire x1="12.3825" y1="6.9875" x2="8.5725" y2="6.9875" width="0.4064" layer="1"/>
+<wire x1="15.3875" y1="6.9875" x2="16.83" y2="6.9875" width="0.4064" layer="16"/>
 <wire x1="16.83" y1="6.9875" x2="20.32" y2="10.4775" width="0.4064" layer="16"/>
-<wire x1="13.6525" y1="6.9875" x2="16.83" y2="6.9875" width="0.4064" layer="1"/>
-<wire x1="16.83" y1="6.9875" x2="20.32" y2="10.4775" width="0.4064" layer="1"/>
+<wire x1="12.3825" y1="6.9875" x2="16.1925" y2="6.9875" width="0.4064" layer="1"/>
 <wire x1="9.99" y1="6.9875" x2="9.99" y2="6.8375" width="0.4064" layer="16"/>
 <wire x1="9.99" y1="6.8375" x2="10.795" y2="6.0325" width="0.4064" layer="16"/>
@@
 <wire x1="8.5725" y1="22.225" x2="7.935" y2="21.5875" width="0.4064" layer="16"/>
 <contactref element="Z1" pad="C"/>
-<contactref element="Z2" pad="C"/>
-<wire x1="16.51" y1="5.2525" x2="16.51" y2="6.35" width="0.4064" layer="16"/>
-<wire x1="16.51" y1="6.35" x2="15.875" y2="6.9875" width="0.4064" layer="16"/>
 <wire x1="6.985" y1="5.2525" x2="8.1075" y2="5.2525" width="0.4064" layer="16"/>
 <wire x1="8.1075" y1="5.2525" x2="9.8425" y2="6.9875" width="0.4064" layer="16"/>
 <wire x1="9.8425" y1="6.9875" x2="9.99" y2="6.9875" width="0.4064" layer="16"/>
+<contactref element="C1" pad="1"/>
+<wire x1="16.1925" y1="6.9875" x2="16.83" y2="6.9875" width="0.4064" layer="1"/>
+<wire x1="16.83" y1="6.9875" x2="20.32" y2="10.4775" width="0.4064" layer="1"/>
 </signal>
 <signal name="SD1">
@@
 <wire x1="3.4925" y1="13.335" x2="3.175" y2="13.0175" width="0.4064" layer="1"/>
 <contactref element="D2" pad="3"/>
-<wire x1="9.8425" y1="8.8875" x2="9.8425" y2="8.89" width="0.4064" layer="1"/>
-<wire x1="9.8425" y1="8.89" x2="11.43" y2="10.4775" width="0.4064" layer="1"/>
-<wire x1="11.43" y1="10.4775" x2="11.43" y2="11.5775" width="0.4064" layer="1"/>
+<wire x1="8.5725" y1="8.8875" x2="9.525" y2="8.89" width="0.4064" layer="1"/>
+<wire x1="9.525" y1="8.89" x2="11.43" y2="10.795" width="0.4064" layer="1"/>
+<wire x1="11.43" y1="10.795" x2="11.43" y2="11.5775" width="0.4064" layer="1"/>
 <wire x1="7.79" y1="7.9375" x2="7.79" y2="9.3775" width="0.4064" layer="16"/>
 <wire x1="7.79" y1="9.3775" x2="8.5725" y2="10.16" width="0.4064" layer="16"/>
@@
 <wire x1="20.0025" y1="13.335" x2="20.32" y2="13.0175" width="0.4064" layer="16"/>
 <contactref element="D4" pad="3"/>
-<wire x1="12.7" y1="11.5775" x2="12.7" y2="10.4775" width="0.4064" layer="1"/>
-<wire x1="12.7" y1="10.4775" x2="13.6525" y2="9.525" width="0.4064" layer="1"/>
-<wire x1="13.6525" y1="9.525" x2="13.6525" y2="8.8875" width="0.4064" layer="1"/>
+<wire x1="12.7" y1="11.5775" x2="12.7" y2="9.525" width="0.4064" layer="1"/>
+<wire x1="12.7" y1="9.525" x2="12.3825" y2="8.8875" width="0.4064" layer="1"/>
 <wire x1="13.1875" y1="7.9375" x2="12.7" y2="7.9375" width="0.4064" layer="16"/>
 <wire x1="12.7" y1="7.9375" x2="12.065" y2="8.5725" width="0.4064" layer="16"/>
